File: pan-tilt-pcb/pan-tilt-pcb_rs485.kicad_sch (KiCad schematic)
At the start: 8 parts, among them U4 ISO1450DW

Commit message: rename to pan-tilt-pcb everywhere
Parts:
- PS1: symbol pan-tilt:CME0303S3C -> pan-tilt-pcb:CME0303S3C
- U4: symbol pan-tilt:ISO1450DW -> pan-tilt-pcb:ISO1450DW
Changed lines of the file:
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@@
 	)
 	(symbol
-		(lib_id "pan-tilt:ISO1450DW")
+		(lib_id "pan-tilt-pcb:ISO1450DW")
 		(at 148.59 110.49 0)
 		(unit 1)
@@
 		)
 		(instances
-			(project ""
+			(project "pan-tilt-pcb"
 				(path "/e3bbbe58-bf8f-42a8-8505-028de8235dc1/98335103-cef0-473f-a7b3-d62ebdf0389c"
 					(reference "U4")
@@
 	)
 	(symbol
-		(lib_id "pan-tilt:CME0303S3C")
+		(lib_id "pan-tilt-pcb:CME0303S3C")
 		(at 148.59 34.29 0)
 		(unit 1)
@@
 		)
 		(instances
-			(project ""
+			(project "pan-tilt-pcb"
 				(path "/e3bbbe58-bf8f-42a8-8505-028de8235dc1/98335103-cef0-473f-a7b3-d62ebdf0389c"
 					(reference "PS1")
@@
 		)
 		(instances
-			(project ""
+			(project "pan-tilt-pcb"
 				(path "/e3bbbe58-bf8f-42a8-8505-028de8235dc1/98335103-cef0-473f-a7b3-d62ebdf0389c"
 					(reference "C24")
@@
 		)
 		(instances
-			(project ""
+			(project "pan-tilt-pcb"
 				(path "/e3bbbe58-bf8f-42a8-8505-028de8235dc1/98335103-cef0-473f-a7b3-d62ebdf0389c"
 					(reference "#FLG06")
@@
 		)
 		(instances
-			(project ""
+			(project "pan-tilt-pcb"
 				(path "/e3bbbe58-bf8f-42a8-8505-028de8235dc1/98335103-cef0-473f-a7b3-d62ebdf0389c"
 					(reference "L2")
@@
 		)
 		(instances
-			(project ""
+			(project "pan-tilt-pcb"
 				(path "/e3bbbe58-bf8f-42a8-8505-028de8235dc1/98335103-cef0-473f-a7b3-d62ebdf0389c"
 					(reference "#PWR057")
